File: io.kicad_sch (KiCad schematic)
At the start: 84 parts, among them J201 USB_microB, J202 DM3BT-DSF-PEJS, J203 USB_A, J204 DM3BT-DSF-PEJS, P201 02x05 Right Angle Shrouded, U201 FT2232HQ, U202 93LC46C-I/MC, U203 TPS2561, U204 MAX3033E, U205 USB3340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

Commit message: Cleaned up the directory and renamed files.  Also converted from the 324 package on the FPGA to the 484 package.  That conversion is still in-progress.
Parts:
- removed U204: MAX3033E, Package_SO:TSSOP-16_4.4x5mm_P0.65mm, symbol myLib:MAX3033E
- added U2: AM26LV31EIPWR, Package_SO:TSSOP-16_4.4x5mm_P0.65mm, symbol Interface:AM26LS31CDB
- C208, C210: JLCPCB Part (none) -> C19666
- C213: JLCPCB Part (none) -> C51412
- C218, C226: value 22µF 10V -> 22µF; JLCPCB Part (none) -> C59461
- C221: footprint Capacitor_Tantalum_SMD:CP_EIA-6032-28_Kemet-C -> Capacitor_SMD:C_Elec_6.3x7.7; FT Rotation Offset (none) -> 180; JLCPCB Part (none) -> C178603; MPN T494C157K010AT -> EEEFTV151XAP; Manu Kemet -> (none)
- C224, C225: JLCPCB Part (none) -> C15849
- D201, D202, D203, D204, D205, D206, D207, D208, D209: JLCPCB Part (none) -> C2297
- FB201, FB202: JLCPCB Part (none) -> C2661452
- J201: JLCPCB Part (none) -> C132560
- J202: value DM3BT-DSF-PEJS -> TF-15x15; footprint Connector_Card:microSD_HC_Hirose_DM3AT-SF-PEJM5 -> Imports:TF15X15; symbol Connector:Micro_SD_Card_Det2 -> myLib:TF-15X15-improved; FT Rotation Offset (none) -> -90; Label (none) -> SD0; MPN DM3AT-SF-PEJM5 -> (none)
- J203: JLCPCB Part (none) -> C599120; MPN 87583-2010BLF -> 87583-3010
- J204: value DM3BT-DSF-PEJS -> TF-15x15; footprint Connector_Card:microSD_HC_Hirose_DM3AT-SF-PEJM5 -> Imports:TF15X15; symbol Connector:Micro_SD_Card_Det2 -> myLib:TF-15X15-improved; FT Rotation Offset (none) -> -90; Label (none) -> SD1; MPN DM3AT-SF-PEJM5 -> (none)
- P201: JLCPCB Part (none) -> C7434504
- R201, R202, R203, R204, R205, R206, R209, R210, R214: value 240 -> 330; MPN RC0603FR-07240RL -> RC0603FR-07330RL
- R224: JLCPCB Part (none) -> C482887
- R232: JLCPCB Part (none) -> C131052
- S201: FT Rotation Offset (none) -> 90; JLCPCB Part (none) -> C319032
- U202: value 93LC46C-I/MC -> 93LC46BT-I/ST; footprint Package_DFN_QFN:DFN-8-1EP_3x2mm_P0.5mm_EP1.75x1.45mm -> Package_SO:TSSOP-8_4.4x3mm_P0.65mm; MPN 93LC46C-I/MC -> 93LC46BC-IST
- U205: FT Rotation Offset (none) -> 180
- Y201: FT Rotation Offset (none) -> -90
Connections:
- net 3V3: now also U2.16 (VDD), U2.4 (G)
- net GND: now also U2.12 (~{G}), U2.8 (GND); no longer J202.10 (DET_A), J204.10 (DET_A)
- net IPblank_N: now also U2.5 (2Z)
- net IPblank_P: now also U2.6 (2Y)
- net IPclk_N: now also U2.3 (1Z)
- net IPclk_P: now also U2.2 (1Y)
- net IPdata_N: now also U2.13 (4Z)
- net IPdata_P: now also U2.14 (4Y)
- net IPlatch_N: now also U2.11 (3Z)
- net IPlatch_P: now also U2.10 (3Y)
- net ip_blank: now also U2.7 (2A)
- net ip_clk: now also U2.1 (1A)
- net ip_data: now also U2.15 (4A)
- net ip_latch: now also U2.9 (3A)
Other:
- moved on the sheet: C220

Commit message: Switched the level converters to 74HCT2G04 and 75LVC2G04.  Still need to remap the FPGA pins to the signal odering.
Other:
- company: (none) -> Vintage Computer Enterprises
Changed lines of the file:
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@@
 	(title_block
 		(title "QSIC - QBUS Storage & I/O Card")
-		(date "2025-03-28")
+		(date "2025-04-12")
 		(rev "0.4")
+		(company "Vintage Computer Enterprises")
 	)
 	(junction
