File: qbus.kicad_sch (KiCad schematic)
At the start: 84 parts, among them J201 USB_microB, J202 DM3BT-DSF-PEJS, J203 USB_A, J204 DM3BT-DSF-PEJS, P201 02x05 Right Angle Shrouded, U201 FT2232HQ, U202 93LC46C-I/MC, U203 TPS2561, U204 MAX3033E, U205 USB3340, X201 ASE-24.000MHz, Y201 12 MHz

Commit message: Cleaned up the directory and renamed files.  Also all the changes to move from the 324 package to the 484 (not yet completed).
Parts:
- removed C201, C202, C203, C204, C205, C206, C207, C209, C211, C212, C214, C217, C219, C220, C222, C223, C227: 100nF, Capacitor_SMD:C_0603_1608Metric, symbol Device:C_Small
- removed C208, C210: 4.7µF 6.3V, Capacitor_SMD:C_0603_1608Metric, symbol Device:C_Polarized_Small_US
- removed C213: 3.3µF 6.3V, Capacitor_SMD:C_0603_1608Metric, symbol Device:C_Small
- removed C215, C216: 8pF, Capacitor_SMD:C_0603_1608Metric, symbol Device:C_Small
- removed C218, C226: 22µF 10V, Capacitor_SMD:C_0603_1608Metric, symbol Device:C_Small
- removed C221: 150µF 10V, Capacitor_Tantalum_SMD:CP_EIA-6032-28_Kemet-C, symbol Device:C_Polarized_Small_US
- removed C224, C225: 1µF, Capacitor_SMD:C_0603_1608Metric, symbol Device:C_Small
- removed C228: 10nF, Capacitor_SMD:C_0603_1608Metric, symbol Device:C_Small
- removed D201, D202, D203, D204, D205, D206, D207, D208, D209: green, LED_SMD:LED_0603_1608Metric, symbol Device:LED_Small_Filled
- removed FB201, FB202: 220Ω @ 100MHz 50mΩ, Inductor_SMD:L_0805_2012Metric, symbol Device:FerriteBead_Small
- removed J201: USB_microB, Connector_USB:USB_Micro-B_Molex_47346-0001, symbol Connector:USB_B_Micro
- removed J202, J204: DM3BT-DSF-PEJS, Connector_Card:microSD_HC_Hirose_DM3AT-SF-PEJM5, symbol Connector:Micro_SD_Card_Det2
- removed J203: USB_A, myMods:Amphenol_87583_USB_A, symbol Connector:USB_A
- removed P201: 02x05 Right Angle Shrouded, myMods:Box_Header_2x05_P2.54mm, symbol Connector_Generic:Conn_02x05_Odd_Even
- removed R201, R202, R203, R204, R205, R206, R209, R210, R214: 240, Resistor_SMD:R_0603_1608Metric, symbol Device:R
- removed R207: 1k, Resistor_SMD:R_0603_1608Metric, symbol Device:R
- removed R208: 12k 1%, Resistor_SMD:R_0603_1608Metric, symbol Device:R
- removed R211, R212, R213: 10k, Resistor_SMD:R_0603_1608Metric, symbol Device:R
- removed R215: 2.2k, Resistor_SMD:R_0603_1608Metric, symbol Device:R
- removed R216, R217: 100k, Resistor_SMD:R_0603_1608Metric, symbol Device:R
- removed R218, R226: 4.7, Resistor_SMD:R_0603_1608Metric, symbol Device:R
- removed R219, R220, R221, R222, R223, R227, R228, R229, R230, R231: 50k, Resistor_SMD:R_0603_1608Metric, symbol Device:R
- removed R224: 56.2k 1%, Resistor_SMD:R_0603_1608Metric, symbol Device:R
- removed R225: 20k, Resistor_SMD:R_0603_1608Metric, symbol Device:R
- removed R232: 8.06k 1%, Resistor_SMD:R_0603_1608Metric, symbol Device:R
- removed S201: DIP Switch x8, Button_Switch_SMD:SW_DIP_SPSTx08_Slide_Omron_A6S-810x_W8.9mm_P2.54mm, symbol myLib:DIP-Switch-8
- removed U201: FT2232HQ, Package_DFN_QFN:QFN-64-1EP_9x9mm_P0.5mm_EP4.35x4.35mm_ThermalVias, symbol myLib:FT2232HQ
- removed U202: 93LC46C-I/MC, Package_DFN_QFN:DFN-8-1EP_3x2mm_P0.5mm_EP1.75x1.45mm, symbol Memory_EEPROM:93CxxC
- removed U203: TPS2561, Package_SON:VSON-10-1EP_3x3mm_P0.5mm_EP1.65x2.4mm_ThermalVias, symbol Interface_USB:TPS2561
- removed U204: MAX3033E, Package_SO:TSSOP-16_4.4x5mm_P0.65mm, symbol myLib:MAX3033E
- removed U205: USB3340, Package_DFN_QFN:QFN-32-1EP_5x5mm_P0.5mm_EP3.3x3.3mm, symbol myLib:USB3340
- removed X201: ASE-24.000MHz, Oscillator:Oscillator_SMD_Abracon_ASE-4Pin_3.2x2.5mm, symbol Oscillator:ASE-xxxMHz
- removed Y201: 12 MHz, Crystal:Crystal_SMD_Abracon_ABM10-4Pin_2.5x2.0mm, symbol Device:Crystal_GND24
- added C401, C402, C403, C404, C405, C406, C407, C408, C409, C410, C411, C412, C413, C414, C415, C416, C417, C418, C419, C420, C421, C422, C423, C424, C425, C426, C427, C428, C429, C430, C431, C432, C433: 100nF, Capacitor_SMD:C_0603_1608Metric, symbol Device:C
- added J401: QBUS_A, DEC:DEC_Edge_Fingers_single_height, symbol DEC:QBUS_A
- added J402: QBUS_B, DEC:DEC_Edge_Fingers_single_height, symbol DEC:QBUS_B
- added R401, R402, R403, R404: 330, Resistor_SMD:R_0603_1608Metric, symbol Device:R
- added R405, R406, R407, R408: 680, Resistor_SMD:R_0603_1608Metric, symbol Device:R
- added RN401, RN402, RN403, RN404: 330/680, Resistor_THT:R_Array_SIP12, symbol Device:R_Network_Dividers_x10_SIP
- added U401, U402, U407, U408, U409, U410, U415, U416, U418, U419, U422: DS8641-LR, Package_DIP:DIP-16_W7.62mm, symbol myLib:DS8641-LR
- added U403, U404, U405, U406, U411, U412, U413, U414, U417, U420, U421: 74LVC8T245, Package_SO:TSSOP-24_4.4x7.8mm_P0.65mm, symbol myLib:74LVC8T245
Connections:
- net 3V3: now also C423.1, C424.1, C425.1, C426.1, C427.1, C428.1, C429.1, C430.1, C431.1, C432.1, C433.1, U403.1 (VCCa), U403.2 (A->B), U404.1 (VCCa), U405.1 (VCCa), U405.2 (A->B), U406.1 (VCCa), U411.1 (VCCa), U411.2 (A->B), U412.1 (VCCa), U413.1 (VCCa), U413.2 (A->B), U414.1 (VCCa), U417.1 (VCCa), U420.1 (VCCa), U420.2 (A->B), U421.1 (VCCa)
- net 5V0: now also C401.1, C402.1, C403.1, C404.1, C405.1, C406.1, C407.1, C408.1, C409.1, C410.1, C411.1, C412.1, C413.1, C414.1, C415.1, C416.1, C417.1, C418.1, C419.1, C420.1, C421.1, C422.1, J401.A2 (+5V), J401.D2 (+5v), J402.A2 (+5V), J402.V1 (+5V), R401.1, R402.1, R403.1, R404.1, RN401.12 (COM2), RN402.12 (COM2), RN403.12 (COM2), RN404.12 (COM2), U401.16 (VCC), U402.16 (VCC), U403.23 (VCCb), U403.24 (VCCb), U404.23 (VCCb), U404.24 (VCCb), U405.23 (VCCb), U405.24 (VCCb), U406.23 (VCCb), U406.24 (VCCb), U407.16 (VCC), U408.16 (VCC), U409.16 (VCC), U410.16 (VCC), U411.23 (VCCb), U411.24 (VCCb), U412.23 (VCCb), U412.24 (VCCb), U413.23 (VCCb), U413.24 (VCCb), U414.23 (VCCb), U414.24 (VCCb), U415.16 (VCC), U416.16 (VCC), U417.23 (VCCb), U417.24 (VCCb), U418.16 (VCC), U419.16 (VCC), U420.23 (VCCb), U420.24 (VCCb), U421.23 (VCCb), U421.24 (VCCb), U422.16 (VCC)
- net GND: now also C401.2, C402.2, C403.2, C404.2, C405.2, C406.2, C407.2, C408.2, C409.2, C410.2, C411.2, C412.2, C413.2, C414.2, C415.2, C416.2, C417.2, C418.2, C419.2, C420.2, C421.2, C422.2, C423.2, C424.2, C425.2, C426.2, C427.2, C428.2, C429.2, C430.2, C431.2, C432.2, C433.2, J401.C2 (GND), J401.J1 (GND), J401.M1 (GND), J401.T1 (GND), J402.C2 (GND), J402.J1 (GND), J402.M1 (GND), J402.T1 (GND), R405.2, R406.2, R407.2, R408.2, RN401.1 (COM1), RN402.1 (COM1), RN403.1 (COM1), RN404.1 (COM1), U401.7 (disB), U401.8 (GND), U401.9 (disA), U402.8 (GND), U402.9 (disA), U403.11 (GND), U403.12 (GND), U403.13 (GND), U403.22 (~{OE}), U404.11 (GND), U404.12 (GND), U404.13 (GND), U404.2 (A->B), U404.22 (~{OE}), U405.11 (GND), U405.12 (GND), U405.13 (GND), U405.22 (~{OE}), U406.11 (GND), U406.12 (GND), U406.13 (GND), U406.2 (A->B), U407.14 (in1), U407.7 (disB), U407.8 (GND), U407.9 (disA), U408.8 (GND), U408.9 (disA), U409.11 (in2), U409.14 (in1), U409.7 (disB), U409.8 (GND), U409.9 (disA), U410.8 (GND), U410.9 (disA), U411.11 (GND), U411.12 (GND), U411.13 (GND), U411.22 (~{OE}), U412.11 (GND), U412.12 (GND), U412.13 (GND), U412.2 (A->B), U412.22 (~{OE}), U413.11 (GND), U413.12 (GND), U413.13 (GND), U413.22 (~{OE}), U414.11 (GND), U414.12 (GND), U414.13 (GND), U414.2 (A->B), U415.8 (GND), U415.9 (disA), U416.14 (in1), U416.7 (disB), U416.8 (GND), U416.9 (disA), U417.11 (GND), U417.12 (GND), U417.13 (GND), U417.2 (A->B), U417.22 (~{OE}), U418.8 (GND), U418.9 (disA), U419.11 (in2), U419.2 (in3), U419.7 (disB), U419.8 (GND), U419.9 (disA), U420.11 (GND), U420.12 (GND), U420.13 (GND), U420.22 (~{OE}), U421.11 (GND), U421.12 (GND), U421.13 (GND), U421.2 (A->B), U422.8 (GND), U422.9 (disA)
- new net: U401.10 (out2), U404.18 (B3)
- new net: U401.11 (in2), U403.18 (B3)
- new net: U401.13 (out1), U404.19 (B2)
- new net: U401.14 (in1), U403.19 (B2)
- new net: U401.2 (in3), U403.20 (B1)
- new net: U401.3 (out3), U404.20 (B1)
- new net: U401.5 (in4), U403.21 (B0)
- new net: U401.6 (out4), U404.21 (B0)
- new net: U404.14 (B7), U407.10 (out2)
- new net: U403.14 (B7), U407.11 (in2)
- new net: U404.15 (B6), U407.13 (out1)
- new net: U403.15 (B6), U407.2 (in3)
- new net: U404.16 (B5), U407.3 (out3)
- new net: U403.16 (B5), U407.5 (in4)
- new net: U404.17 (B4), U407.6 (out4)
- new net: U412.14 (B7), U416.10 (out2)
- new net: U412.15 (B6), U416.13 (out1)
- new net: U412.17 (B4), U416.6 (out4)
- new net: U409.10 (out2), U412.18 (B3)
- new net: U409.13 (out1), U412.19 (B2)
- new net: U409.3 (out3), U412.20 (B1)
- new net: U409.6 (out4), U412.21 (B0)
- new net: U409.2 (in3), U411.20 (B1)
- new net: U409.5 (in4), U411.21 (B0)
- new net: U411.17 (B4), U416.11 (in2)
- new net: U411.18 (B3), U416.2 (in3)
- new net: U411.19 (B2), U416.5 (in4)
- new net: U402.10 (out2), U406.18 (B3)
- new net: U402.11 (in2), U405.18 (B3)
- new net: U402.13 (out1), U406.19 (B2)
- new net: U402.14 (in1), U405.19 (B2)
- new net: U402.2 (in3), U405.20 (B1)
- new net: U402.3 (out3), U406.20 (B1)
- new net: U402.5 (in4), U405.21 (B0)
- new net: U402.6 (out4), U406.21 (B0)
- new net: U405.14 (B7), U408.11 (in2)
- new net: U405.15 (B6), U408.14 (in1)
- new net: U405.16 (B5), U408.2 (in3)
- new net: U405.17 (B4), U408.5 (in4)
- new net: U406.14 (B7), U408.10 (out2)
- new net: U406.15 (B6), U408.13 (out1)
- new net: U406.16 (B5), U408.3 (out3)
- new net: U406.17 (B4), U408.6 (out4)
- new net: U410.10 (out2), U414.18 (B3)
- new net: U410.11 (in2), U413.18 (B3)
- new net: U410.13 (out1), U414.19 (B2)
- new net: U410.14 (in1), U413.19 (B2)
- new net: U410.2 (in3), U413.20 (B1)
- new net: U410.3 (out3), U414.20 (B1)
- new net: U410.5 (in4), U413.21 (B0)
- new net: U410.6 (out4), U414.21 (B0)
- new net: U413.14 (B7), U415.11 (in2)
- new net: U413.15 (B6), U415.14 (in1)
- new net: U413.16 (B5), U415.2 (in3)
- new net: U413.17 (B4), U415.5 (in4)
- new net: U414.14 (B7), U415.10 (out2)
- new net: U414.15 (B6), U415.13 (out1)
- new net: U414.16 (B5), U415.3 (out3)
- new net: U414.17 (B4), U415.6 (out4)
- new net: U420.14 (B7), U422.11 (in2)
- new net: U420.15 (B6), U422.14 (in1)
- new net: U420.16 (B5), U422.2 (in3)
- new net: U420.17 (B4), U422.5 (in4)
- new net: U418.11 (in2), U420.18 (B3)
- new net: U418.14 (in1), U420.19 (B2)
- new net: U418.2 (in3), U420.20 (B1)
- new net: U418.5 (in4), U420.21 (B0)
- new net: U421.14 (B7), U422.10 (out2)
- new net: U421.15 (B6), U422.13 (out1)
- new net: U421.16 (B5), U422.3 (out3)
- new net: U421.17 (B4), U422.6 (out4)
- new net: U418.10 (out2), U421.18 (B3)
- new net: U418.13 (out1), U421.19 (B2)
- new net: U418.3 (out3), U421.20 (B1)
- new net: U418.6 (out4), U421.21 (B0)
- new net: U411.14 (B7), U419.14 (in1)
- new net: U411.15 (B6), U419.5 (in4)
- new net: U417.18 (B3), U419.10 (out2)
- new net: U417.19 (B2), U419.13 (out1)
- new net: U417.20 (B1), U419.3 (out3)
- new net: U417.21 (B0), U419.6 (out4)
- new net BBS7: J401.P2 (BBS7), RN402.11 (R10), U402.12 (bus2)
- new net BDAL0: J401.U2 (BDAL0), RN402.6 (R5), U408.1 (bus3)
- new net BDAL1: J401.V2 (BDAL1), RN402.5 (R4), U408.4 (bus4)
- new net BDAL10: J402.P2 (BDAL10), RN404.7 (R6), U418.12 (bus2)
- new net BDAL11: J402.R2 (BDAL11), RN404.6 (R5), U418.15 (bus1)
- new net BDAL12: J402.S2 (BDAL12), RN404.5 (R4), U422.1 (bus3)
- new net BDAL13: J402.T2 (BDAL13), RN404.4 (R3), U422.4 (bus4)
- new net BDAL14: J402.U2 (BDAL14), RN404.3 (R2), U422.12 (bus2)
- new net BDAL15: J402.V2 (BDAL15), RN404.2 (R1), U422.15 (bus1)
- new net BDAL16: J401.C1 (BDAL16), RN401.7 (R6), U402.1 (bus3)
- new net BDAL17: J401.D1 (BDAL17), RN401.6 (R5), U402.4 (bus4)
- new net BDAL18: J402.C1 (BDAL18), RN402.2 (R1), U408.15 (bus1)
- new net BDAL19: J402.D1 (BDAL19), RN403.11 (R10), U408.12 (bus2)
- new net BDAL2: J402.E2 (BDAL2), RN403.9 (R8), U410.1 (bus3)
- new net BDAL20: J402.E1 (BDAL20), RN403.10 (R9), U410.4 (bus4)
- new net BDAL21: J402.F1 (BDAL21), RN403.4 (R3), U410.15 (bus1)
- new net BDAL3: J402.F2 (BDAL3), RN403.5 (R4), U410.12 (bus2)
- new net BDAL4: J402.H2 (BDAL4), RN403.3 (R2), U415.1 (bus3)
- new net BDAL5: J402.J2 (BDAL5), RN403.2 (R1), U415.4 (bus4)
- new net BDAL6: J402.K2 (BDAL6), RN404.11 (R10), U415.12 (bus2)
- new net BDAL7: J402.L2 (BDAL7), RN404.10 (R9), U415.15 (bus1)
- new net BDAL8: J402.M2 (BDAL8), RN404.9 (R8), U418.1 (bus3)
- new net BDAL9: J402.N2 (BDAL9), RN404.8 (R7), U418.4 (bus4)
- new net BDCOK: J402.A1 (BDCOK), RN402.4 (R3), U416.15 (bus1)
- new net BDIN: J401.H2 (BDIN), RN401.5 (R4), U407.1 (bus3)
- new net BDMGI: J401.R2 (BDMGI), R403.2, R407.1, U409.15 (bus1)
- new net BDMGO: J401.S2 (BDMGO), R404.2, R408.1, U416.1 (bus3)
- new net BDMR: J401.N1 (BDMR), RN402.10 (R9), U409.1 (bus3)
- new net BDOUT: J401.E2 (BDOUT), RN401.9 (R8), U401.12 (bus2)
- new net BEVNT: J402.R1 (BEVNT), RN403.6 (R5), U419.12 (bus2)
- new net BHALT: J401.P1 (BHALT), RN402.9 (R8), U409.12 (bus2)
- new net BIAKI: J401.M2 (BIAKI), R401.2, R405.1, U407.15 (bus1)
- new net BIAKO: J401.N2 (BIAKO), R402.2, R406.1, U409.4 (bus4)
- new net BINIT: J401.T2 (BINIT), RN402.7 (R6), U416.12 (bus2)
- new net BIRQ4: J401.L2 (BIRQ4), RN401.3 (R2), U407.12 (bus2)
- new net BIRQ5: J401.A1 (BIRQ5), RN401.11 (R10), U401.1 (bus3)
- new net BIRQ6: J401.B1 (BIRQ6), RN401.10 (R9), U401.4 (bus4)
- new net BIRQ7: J402.P1 (BIRQ7), RN403.7 (R6), U419.15 (bus1)
- new net BPOK: J402.B1 (BPOK), RN402.3 (R2), U419.1 (bus3)
- new net BREF: J401.R1 (BREF), RN402.8 (R7), U416.4 (bus4)
- new net BRPLY: J401.F2 (BRPLY), RN401.8 (R7), U401.15 (bus1)
- new net BSACK: J402.N1 (BSACK), RN403.8 (R7), U419.4 (bus4)
- new net BSYNC: J401.J2 (BSYNC), RN401.4 (R3), U407.4 (bus4)
- new net BWTBT: J401.K2 (BWTBT), RN401.2 (R1), U402.15 (bus1)
- new net RDCOK: U412.9 (A6)
- new net RDIN: U404.8 (A5)
- new net RDMGI: U412.5 (A2)
- new net RDMR: U412.4 (A1)
- new net RDOUT: U404.6 (A3)
- new net REVNT: U417.6 (A3)
- new net RHALT: U412.6 (A3)
- new net RIAKI: U404.9 (A6)
- new net RINIT: U412.10 (A7)
- new net RIRQ4: U404.10 (A7)
- new net RIRQ5: U404.4 (A1)
- new net RIRQ6: U404.3 (A0)
- new net RIRQ7: U417.5 (A2)
- new net RPOK: U417.4 (A1)
- new net RREF: U412.7 (A4)
- new net RRPLY: U404.5 (A2)
- new net RSACK: U417.3 (A0)
- new net RSYNC: U404.7 (A4)
- new net TDIN: U403.9 (A6)
- new net TDMGO: U411.6 (A3)
- new net TDMR: U411.4 (A1)
- new net TDOUT: U403.6 (A3)
- new net TIAKO: U411.3 (A0)
- new net TINIT: U411.7 (A4)
- new net TIRQ4: U403.10 (A7)
- new net TIRQ5: U403.4 (A1)
- new net TIRQ6: U403.3 (A0)
- new net TIRQ7: U411.10 (A7)
- new net TREF: U411.5 (A2)
- new net TRPLY: U403.5 (A2)
- new net TSACK: U411.9 (A6)
- new net TSYNC: U403.8 (A5)
- new net ZBS7: U405.6 (A3), U406.6 (A3)
- new net ZDAL0: U405.8 (A5), U406.8 (A5)
- new net ZDAL1: U405.7 (A4), U406.7 (A4)
- new net ZDAL10: U420.6 (A3), U421.6 (A3)
- new net ZDAL11: U420.5 (A2), U421.5 (A2)
- new net ZDAL12: U420.8 (A5), U421.8 (A5)
- new net ZDAL13: U420.7 (A4), U421.7 (A4)
- new net ZDAL14: U420.10 (A7), U421.10 (A7)
- new net ZDAL15: U420.9 (A6), U421.9 (A6)
- new net ZDAL16: U405.4 (A1), U406.4 (A1)
- new net ZDAL17: U405.3 (A0), U406.3 (A0)
- new net ZDAL18: U405.9 (A6), U406.9 (A6)
- new net ZDAL19: U405.10 (A7), U406.10 (A7)
- new net ZDAL2: U413.4 (A1), U414.4 (A1)
- new net ZDAL20: U413.3 (A0), U414.3 (A0)
- new net ZDAL21: U413.5 (A2), U414.5 (A2)
- new net ZDAL3: U413.6 (A3), U414.6 (A3)
- new net ZDAL4: U413.8 (A5), U414.8 (A5)
- new net ZDAL5: U413.7 (A4), U414.7 (A4)
- new net ZDAL6: U413.10 (A7), U414.10 (A7)
- new net ZDAL7: U413.9 (A6), U414.9 (A6)
- new net ZDAL8: U420.4 (A1), U421.4 (A1)
- new net ZDAL9: U420.3 (A0), U421.3 (A0)
- new net ZWTBT: U405.5 (A2), U406.5 (A2)
- new net ~{RxDAL}: U406.22 (~{OE}), U414.22 (~{OE}), U421.22 (~{OE})
- new net ~{TxDAL_5}: U402.7 (disB), U408.7 (disB), U410.7 (disB), U411.16 (B5), U415.7 (disB), U418.7 (disB), U422.7 (disB)
- new net ~{TxDAL}: U411.8 (A5)
- no-connect marks 29 -> 30
Other:
- note added: "Optional Bus Terminators"
- company: (none) -> Vintage Computer Engineering

Commit message: Cleaned up the directory and renamed files.  Also converted from the 324 package on the FPGA to the 484 package.  That conversion is still in-progress.
Parts:
- added C1, C2, C3, C4: 10 uF 16V, Capacitor_Tantalum_SMD:CP_EIA-3216-18_Kemet-A, symbol Device:C_Polarized_Small_US
- RN401, RN402, RN403, RN404: now not fitted; now left out of the parts list
Connections:
- net ~{RxDAL} is gone; now on net GND: U406.22 (~{OE}), U414.22 (~{OE}), U421.22 (~{OE})
- net 5V0: now also C1.1, C2.1, C3.1, C4.1
- net GND: now also U402.7 (disB), U408.7 (disB), U410.7 (disB), U415.7 (disB), U418.7 (disB), U422.7 (disB), C1.2, C2.2, C3.2, C4.2
- net ZBS7 renamed RBS7
- net RBS7: no longer U405.6 (A3)
- net ZDAL0 renamed RDAL0
- net RDAL0: no longer U405.8 (A5)
- net ZDAL1 renamed RDAL1
- net RDAL1: no longer U405.7 (A4)
- net ZDAL10 renamed RDAL10
- net RDAL10: no longer U420.6 (A3)
- net ZDAL11 renamed RDAL11
- net RDAL11: no longer U420.5 (A2)
- net ZDAL12 renamed RDAL12
- net RDAL12: no longer U420.8 (A5)
- net ZDAL13 renamed RDAL13
- net RDAL13: no longer U420.7 (A4)
- net ZDAL14 renamed RDAL14
- net RDAL14: no longer U420.10 (A7)
- net ZDAL15 renamed RDAL15
- net RDAL15: no longer U420.9 (A6)
- net ZDAL16 renamed RDAL16
- net RDAL16: no longer U405.4 (A1)
- net ZDAL17 renamed RDAL17
- net RDAL17: no longer U405.3 (A0)
- net ZDAL18 renamed RDAL18
- net RDAL18: no longer U405.9 (A6)
- net ZDAL19 renamed RDAL19
- net RDAL19: no longer U405.10 (A7)
- net ZDAL2 renamed RDAL2
- net RDAL2: no longer U413.4 (A1)
- net ZDAL20 renamed RDAL20
- net RDAL20: no longer U413.3 (A0)
- net ZDAL21 renamed RDAL21
- net RDAL21: no longer U413.5 (A2)
- net ZDAL3 renamed RDAL3
- net RDAL3: no longer U413.6 (A3)
- net ZDAL4 renamed RDAL4
- net RDAL4: no longer U413.8 (A5)
- net ZDAL5 renamed RDAL5
- net RDAL5: no longer U413.7 (A4)
- net ZDAL6 renamed RDAL6
- net RDAL6: no longer U413.10 (A7)
- net ZDAL7 renamed RDAL7
- net RDAL7: no longer U413.9 (A6)
- net ZDAL8 renamed RDAL8
- net RDAL8: no longer U420.4 (A1)
- net ZDAL9 renamed RDAL9
- net RDAL9: no longer U420.3 (A0)
- net ZWTBT renamed RWTBT
- net RWTBT: no longer U405.5 (A2)
- removed net ~{TxDAL_5}: U402.7 (disB), U408.7 (disB), U410.7 (disB), U411.16 (B5), U415.7 (disB), U418.7 (disB), U422.7 (disB)
- net ~{TxDAL}: no longer names the net of U411.8 (A5)
- new net TBS7: U405.6 (A3)
- new net TDAL0: U405.8 (A5)
- new net TDAL1: U405.7 (A4)
- new net TDAL10: U420.6 (A3)
- new net TDAL11: U420.5 (A2)
- new net TDAL12: U420.8 (A5)
- new net TDAL13: U420.7 (A4)
- new net TDAL14: U420.10 (A7)
- new net TDAL15: U420.9 (A6)
- new net TDAL16: U405.4 (A1)
- new net TDAL17: U405.3 (A0)
- new net TDAL18: U405.9 (A6)
- new net TDAL19: U405.10 (A7)
- new net TDAL2: U413.4 (A1)
- new net TDAL20: U413.3 (A0)
- new net TDAL21: U413.5 (A2)
- new net TDAL3: U413.6 (A3)
- new net TDAL4: U413.8 (A5)
- new net TDAL5: U413.7 (A4)
- new net TDAL6: U413.10 (A7)
- new net TDAL7: U413.9 (A6)
- new net TDAL8: U420.4 (A1)
- new net TDAL9: U420.3 (A0)
- new net TWTBT: U405.5 (A2)
- no-connect marks 30 -> 32

Commit message: Switched the level converters to 74HCT2G04 and 75LVC2G04.  Still need to remap the FPGA pins to the signal odering.
Parts:
- removed C412, C413, C414, C415, C416, C417, C418, C419, C420, C421, C422, C423, C424, C425, C426, C427, C428, C429, C430, C431, C432, C433: 100nF, Capacitor_SMD:C_0603_1608Metric, symbol Device:C
- removed U403, U404, U405, U406, U411, U412, U413, U414, U417, U420, U421: 74LVC8T245, Package_SO:TSSOP-24_4.4x7.8mm_P0.65mm, symbol myLib:74LVC8T245
- added U10, U11, U12, U13, U14, U27, U3, U34, U38, U4, U40, U44, U46, U48, U5, U50, U52, U6, U7, U8, U9: 74LVC2GU04, Package_TO_SOT_SMD:SOT-363_SC-70-6, symbol myLib:74LVC2G04
- added U15, U16, U17, U18, U19, U20, U21, U22, U23, U24, U25, U26, U28, U29, U30, U32, U33, U35, U36, U41: 74HCT2GU04, Package_TO_SOT_SMD:SOT-363_SC-70-6, symbol myLib:74LVC2G04
- J401: footprint DEC:DEC_Edge_Fingers_single_height -> myMods:DEC_Edge_Fingers_single_height-1; symbol DEC:QBUS_A -> myLib:QBUS_A; slot (none) -> A
- J402: footprint DEC:DEC_Edge_Fingers_single_height -> myMods:DEC_Edge_Fingers_single_height-1; symbol DEC:QBUS_B -> myLib:QBUS_B; slot (none) -> B
Connections:
- net GND: now also U30.1, U35.1
- net RBS7: now also U3.4
- net RDAL0: now also U6.6
- net RDAL1: now also U6.4
- net RDAL10: now also U11.4
- net RDAL11: now also U11.6
- net RDAL12: now also U14.6
- net RDAL13: now also U14.4
- net RDAL14: now also U13.4
- net RDAL15: now also U13.6
- net RDAL16: now also U4.6
- net RDAL17: now also U4.4
- net RDAL18: now also U5.6
- net RDAL19: now also U5.4
- net RDAL2: now also U8.6
- net RDAL20: now also U8.4
- net RDAL21: now also U7.6
- net RDAL3: now also U7.4
- net RDAL4: now also U10.6
- net RDAL5: now also U10.4
- net RDAL6: now also U9.4
- net RDAL7: now also U9.6
- net RDAL8: now also U12.6
- net RDAL9: now also U12.4
- net RDCOK: now also U46.6
- net RDIN: now also U40.6
- net RDMGI: now also U48.4
- net RDMR: now also U44.4
- net RDOUT: now also U27.4
- net REVNT: now also U50.4
- net RHALT: now also U44.6
- net RIAKI: now also U38.6
- net RINIT: now also U46.4
- net RIRQ4: now also U38.4
- net RIRQ5: now also U34.6
- net RIRQ6: now also U34.4
- net RIRQ7: now also U50.6
- net RPOK: now also U52.4
- net RREF: now also U48.6
- net RRPLY: now also U27.6
- net RSACK: now also U52.6
- net RSYNC: now also U40.4
- net RWTBT: now also U3.6
- net TBS7: now also U15.3
- net TDAL0: now also U18.1
- net TDAL1: now also U18.3
- net TDAL10: now also U23.3
- net TDAL11: now also U23.1
- net TDAL12: now also U26.1
- net TDAL13: now also U26.3
- net TDAL14: now also U25.3
- net TDAL15: now also U25.1
- net TDAL16: now also U16.1
- net TDAL17: now also U16.3
- net TDAL18: now also U17.1
- net TDAL19: now also U17.3
- net TDAL2: now also U20.1
- net TDAL20: now also U20.3
- net TDAL21: now also U19.1
- net TDAL3: now also U19.3
- net TDAL4: now also U22.1
- net TDAL5: now also U22.3
- net TDAL6: now also U21.3
- net TDAL7: now also U21.1
- net TDAL8: now also U24.1
- net TDAL9: now also U24.3
- net TDIN: now also U32.1
- net TDMR: now also U33.1
- net TDOUT: now also U28.3
- net TIAKO: now also U33.3
- net TINIT: now also U35.3
- net TIRQ4: now also U30.3
- net TIRQ5: now also U29.1
- net TIRQ6: now also U29.3
- net TIRQ7: now also U41.3
- net TRPLY: now also U28.1
- net TSACK: now also U41.1
- net TSYNC: now also U32.3
- net TWTBT: now also U15.1
- net at U401.10 (out2): now also U27.3
- net at U401.11 (in2): now also U28.4
- net at U401.13 (out1): now also U27.1
- net at U401.14 (in1): now also U28.6
- net at U401.2 (in3): now also U29.6
- net at U401.3 (out3): now also U34.1
- net at U401.5 (in4): now also U29.4
- net at U401.6 (out4): now also U34.3
- net at U407.10 (out2): now also U38.3
- net at U407.11 (in2): now also U30.4
- net at U407.13 (out1): now also U38.1
- net at U407.2 (in3): now also U32.6
- net at U407.3 (out3): now also U40.1
- net at U407.5 (in4): now also U32.4
- net at U407.6 (out4): now also U40.3
- net at U416.10 (out2): now also U46.3
- net at U416.13 (out1): now also U46.1
- net at U416.6 (out4): now also U48.1
- net at U409.10 (out2): now also U44.1
- net at U409.13 (out1): now also U48.3
- net at U409.3 (out3): now also U44.3
- net at U409.2 (in3): now also U33.6
- net at U409.5 (in4): now also U33.4
- net at U416.11 (in2): now also U35.4
- net at U416.2 (in3): now also U36.6
- net at U416.5 (in4): now also U36.4
- net at U402.10 (out2): now also U3.3
- net at U402.11 (in2): now also U15.4
- net at U402.13 (out1): now also U3.1
- net at U402.14 (in1): now also U15.6
- net at U402.2 (in3): now also U16.6
- net at U402.3 (out3): now also U4.1
- net at U402.5 (in4): now also U16.4
- net at U402.6 (out4): now also U4.3
- net at U408.11 (in2): now also U17.4
- net at U408.14 (in1): now also U17.6
- net at U408.2 (in3): now also U18.6
- net at U408.5 (in4): now also U18.4
- net at U408.10 (out2): now also U5.3
- net at U408.13 (out1): now also U5.1
- net at U408.3 (out3): now also U6.1
- net at U408.6 (out4): now also U6.3
- net at U410.10 (out2): now also U7.3
- net at U410.11 (in2): now also U19.4
- net at U410.13 (out1): now also U7.1
- net at U410.14 (in1): now also U19.6
- net at U410.2 (in3): now also U20.6
- net at U410.3 (out3): now also U8.1
- net at U410.5 (in4): now also U20.4
- net at U410.6 (out4): now also U8.3
- net at U415.11 (in2): now also U21.4
- net at U415.14 (in1): now also U21.6
- net at U415.2 (in3): now also U22.6
- net at U415.5 (in4): now also U22.4
- net at U415.10 (out2): now also U9.3
- net at U415.13 (out1): now also U9.1
- net at U415.3 (out3): now also U10.1
- net at U415.6 (out4): now also U10.3
- net at U422.11 (in2): now also U25.4
- net at U422.14 (in1): now also U25.6
- net at U422.2 (in3): now also U26.6
- net at U422.5 (in4): now also U26.4
- net at U418.11 (in2): now also U23.4
- net at U418.14 (in1): now also U23.6
- net at U418.2 (in3): now also U24.6
- net at U418.5 (in4): now also U24.4
- net at U422.10 (out2): now also U13.3
- net at U422.13 (out1): now also U13.1
- net at U422.3 (out3): now also U14.1
- net at U422.6 (out4): now also U14.3
- net at U418.10 (out2): now also U11.3
- net at U418.13 (out1): now also U11.1
- net at U418.3 (out3): now also U12.1
- net at U418.6 (out4): now also U12.3
- net at U419.14 (in1): now also U41.4
- net at U419.5 (in4): now also U41.6
- net at U419.10 (out2): now also U50.3
- net at U419.13 (out1): now also U50.1
- net at U419.3 (out3): now also U52.3
- net at U419.6 (out4): now also U52.1
- no-connect marks 32 -> 20
Other:
- company: Vintage Computer Engineering -> Vintage Computer Enterprises
- moved on the sheet: C401, C402, C403, C404, C405, C406, C407, C408, C409, C410, C411, U401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
