File: qsic.kicad_sch (KiCad schematic)
At the start: 15 parts, among them U101 MT25Q, U102 XC7A75T-1CSG324

Commit message: Cleaned up the directory and renamed files.  Also converted from the 324 package on the FPGA to the 484 package.  That conversion is still in-progress.
Parts:
- removed U102: XC7A75T-1CSG324, Package_BGA:Xilinx_CSG324, symbol FPGA_Xilinx_Artix7:XC7A75T-CSG324
- added C107: 22µF, Capacitor_SMD:C_0603_1608Metric, symbol Device:C_Small
- added U1: XC7A75T-2FGG484, Package_BGA:Xilinx_FGG484, symbol FPGA_Xilinx_Artix7:XC7A75T-FGG484
- C101, C102, C103, C104, C106: value 22µF 10V -> 22µF; JLCPCB Part (none) -> C59461
- D101: JLCPCB Part (none) -> C2297
- R104: value 240 -> 330; MPN RC0603FR-07240RL -> RC0603FR-07330RL
Connections:
- net 3V3: now also C107.2, U1.AA17 (VCCO_13), U1.AA7 (VCCO_34), U1.AB14 (VCCO_13), U1.AB4 (VCCO_34), U1.C1 (VCCO_35), U1.F12 (VCCO_0), U1.F2 (VCCO_35), U1.H6 (VCCO_35), U1.J3 (VCCO_35), U1.M14 (VCCO_14), U1.M4 (VCCO_35), U1.N1 (VCCO_35), U1.P18 (VCCO_14), U1.R15 (VCCO_14), U1.R5 (VCCO_34), U1.T12 (VCCO_0), U1.T2 (VCCO_34), U1.T22 (VCCO_14), U1.U11 (M0_0), U1.U19 (VCCO_14), U1.U8 (CFGBVS_0), U1.V16 (VCCO_13), U1.V6 (VCCO_34), U1.W13 (VCCO_13), U1.W3 (VCCO_34), U1.Y10 (VCCO_13), U1.Y20 (VCCO_14)
- net GND: now also C107.1, U1.L9 (VREFN_0), U1.M10 (VREFP_0), U1.U10 (M1_0), U1.U9 (M2_0)
- net LED_0: now also U1.T18 (IO_L20N_T3_A07_D23_14)
- net LED_1: now also U1.R18 (IO_L20P_T3_A08_D24_14)
- net LED_2: now also U1.V13 (IO_L13P_T2_MRCC_13)
- net LED_3: now also U1.W16 (IO_L16N_T2_13)
- net LED_4: now also U1.U16 (IO_L17N_T2_13)
- net LED_5: now also U1.V15 (IO_L14N_T2_SRCC_13)
- net LED_6: now also U1.T16 (IO_L17P_T2_13)
- net LED_7: now also U1.T14 (IO_L15P_T2_DQS_13)
- net PROG_B: now also U1.N12 (PROGRAM_B_0)
- net RDCOK: now also U1.P2 (IO_L22P_T3_35)
- net RDIN: now also U1.T5 (IO_L14P_T2_SRCC_34)
- net RDMGI: now also U1.R3 (IO_L3P_T0_DQS_34)
- net RDMR: now also U1.T1 (IO_L1P_T0_34)
- net RDOUT: now also U1.Y3 (IO_L9P_T1_DQS_34)
- net REVNT: now also U1.M6 (IO_L23P_T3_35)
- net RHALT: now also U1.R2 (IO_L3N_T0_DQS_34)
- net RIAKI: now also U1.AB2 (IO_L8N_T1_34)
- net RINIT: now also U1.P1 (IO_L20N_T3_35)
- net RIRQ4: now also U1.AB1 (IO_L7N_T1_34)
- net RIRQ5: now also U1.Y4 (IO_L11P_T1_SRCC_34)
- net RIRQ6: now also U1.AB3 (IO_L8P_T1_34)
- net RIRQ7: now also U1.L1 (IO_L15N_T2_DQS_35)
- net RPOK: now also U1.M3 (IO_L16P_T2_35)
- net RREF: now also U1.R1 (IO_L20P_T3_35)
- net RRPLY: now also U1.AA3 (IO_L9N_T1_DQS_34)
- net RSACK: now also U1.M5 (IO_L23N_T3_35)
- net RSYNC: now also U1.V4 (IO_L12P_T1_MRCC_34)
- net RXD: now also U1.Y17 (IO_0_13)
- net SW_0: now also U1.V14 (IO_L13N_T2_MRCC_13)
- net SW_1: now also U1.T15 (IO_L15N_T2_DQS_13)
- net SW_2: now also U1.U15 (IO_L14P_T2_SRCC_13)
- net SW_3: now also U1.W15 (IO_L16P_T2_13)
- net SW_4: now also U1.V17 (IO_L16P_T2_CSI_B_14)
- net SW_5: now also U1.W17 (IO_L16N_T2_A15_D31_14)
- net SW_6: now also U1.V18 (IO_L14P_T2_SRCC_14)
- net SW_7: now also U1.V19 (IO_L14N_T2_SRCC_14)
- net TCK: now also U1.V12 (TCK_0)
- net TDI: now also U1.R13 (TDI_0)
- net TDIN: now also U1.W5 (IO_L15N_T2_DQS_34)
- net TDMGO: now also U1.N2 (IO_L22N_T3_35)
- net TDMR: now also U1.P5 (IO_L21P_T3_DQS_35)
- net TDO: now also U1.U13 (TDO_0)
- net TDOUT: now also U1.AB5 (IO_L10N_T1_34)
- net TIAKO: now also U1.P4 (IO_L21N_T3_DQS_35)
- net TINIT: now also U1.N3 (IO_L19N_T3_VREF_35)
- net TIRQ4: now also U1.AA4 (IO_L11N_T1_SRCC_34)
- net TIRQ5: now also U1.AB6 (IO_L20N_T3_34)
- net TIRQ6: now also U1.AA8 (IO_L22P_T3_34)
- net TIRQ7: now also U1.M2 (IO_L16N_T2_35)
- net TMS: now also U1.T13 (TMS_0)
- net TREF: now also U1.P6 (IO_L24P_T3_35)
- net TRPLY: now also U1.AA6 (IO_L18N_T2_34)
- net TSACK: now also U1.M1 (IO_L15P_T2_DQS_35)
- net TSYNC: now also U1.AA5 (IO_L10P_T1_34)
- net TXD: now also U1.AB17 (IO_L2N_T0_13)
- net ip_blank: now also U1.T20 (IO_L6N_T0_D08_VREF_14)
- net ip_clk: now also U1.AA20 (IO_L8P_T1_D11_14)
- net ip_data: now also U1.W21 (IO_L7P_T1_D09_14)
- net ip_latch: now also U1.W19 (IO_L12P_T1_MRCC_14)
- net sd0_clk: now also U1.U20 (IO_L11P_T1_SRCC_14)
- net sd0_cmd: now also U1.AB22 (IO_L10N_T1_D15_14)
- net sd0_dat0: now also U1.AB21 (IO_L10P_T1_D14_14)
- net sd0_dat1: now also U1.W20 (IO_L12N_T1_MRCC_14)
- net sd0_dat2: now also U1.Y22 (IO_L9N_T1_DQS_D13_14)
- net sd0_dat3: now also U1.AA21 (IO_L8N_T1_D12_14)
- net sd0_det: now also U1.W22 (IO_L7N_T1_D10_14)
- net sd1_clk: now also U1.V20 (IO_L11N_T1_SRCC_14)
- net sd1_cmd: now also U1.N17 (IO_L21P_T3_DQS_14)
- net sd1_dat0: now also U1.W11 (IO_L12P_T1_MRCC_13)
- net sd1_dat1: now also U1.Y12 (IO_L11N_T1_SRCC_13)
- net sd1_dat2: now also U1.P14 (IO_L19P_T3_A10_D26_14)
- net sd1_dat3: now also U1.P15 (IO_L22P_T3_A05_D21_14)
- net sd1_det: now also U1.Y21 (IO_L9P_T1_DQS_14)
- net usb0_clk60: now also U1.U17 (IO_L18P_T2_A12_D28_14)
- net usb0_d0: now also U1.AA19 (IO_L15P_T2_DQS_RDWR_B_14)
- net usb0_d1: now also U1.R14 (IO_L19N_T3_A09_D25_VREF_14)
- net usb0_d2: now also U1.Y18 (IO_L13P_T2_MRCC_14)
- net usb0_d3: now also U1.R16 (IO_L22N_T3_A04_D20_14)
- net usb0_d4: now also U1.Y11 (IO_L11P_T1_SRCC_13)
- net usb0_d5: now also U1.P17 (IO_L21N_T3_DQS_A06_D22_14)
- net usb0_d6: now also U1.W10 (IO_L10N_T1_13)
- net usb0_d7: now also U1.W12 (IO_L12N_T1_MRCC_13)
- net usb0_dir: now also U1.AB18 (IO_L17N_T2_A13_D29_14)
- net usb0_nxt: now also U1.Y19 (IO_L13N_T2_MRCC_14)
- net usb0_reset: now also U1.U18 (IO_L18N_T2_A11_D27_14)
- net usp0_stp: now also U1.AB20 (IO_L15N_T2_DQS_DOUT_CSO_B_14)
- net ~{CTS}: now also U1.AA16 (IO_L1N_T0_13)
- net ~{DCD}: now also U1.AB13 (IO_L3N_T0_DQS_13)
- net ~{DSR}: now also U1.Y13 (IO_L5P_T0_13)
- net ~{DTR}: now also U1.AA15 (IO_L4P_T0_13)
- net ~{RI}: now also U1.AA13 (IO_L3P_T0_DQS_13)
- net ~{RTS}: now also U1.Y16 (IO_L1P_T0_13)
- net at D101.1 (K): now also U1.G11 (DONE_0)
- net at R105.2: now also U1.U12 (INIT_B_0)
- net at R103.2, U101.1 (~{S}): now also U1.T19 (IO_L6P_T0_FCS_B_14)
- net at R101.2, U101.3 (~{W}/DQ2): now also U1.P21 (IO_L2P_T0_D02_14)
- net at R102.2, U101.7 (~{HOLD}/DQ3): now also U1.R21 (IO_L2N_T0_D03_14)
- net at U101.2 (DQ1): now also U1.R22 (IO_L1N_T0_D01_DIN_14)
- net at U101.5 (DQ0): now also U1.P22 (IO_L1P_T0_D00_MOSI_14)
- net at U101.6 (C): now also U1.L12 (CCLK_0)
- new net RBS7: U1.T6 (IO_L17N_T2_34)
- new net RDAL0: U1.U1 (IO_L1N_T0_34)
- new net RDAL1: U1.T4 (IO_L13N_T2_MRCC_34)
- new net RDAL10: U1.F1 (IO_L5N_T0_AD13N_35)
- new net RDAL11: U1.G3 (IO_L11N_T1_SRCC_35)
- new net RDAL12: U1.E1 (IO_L3P_T0_DQS_AD5P_35)
- new net RDAL13: U1.G4 (IO_L12N_T1_MRCC_35)
- new net RDAL14: U1.D1 (IO_L3N_T0_DQS_AD5N_35)
- new net RDAL15: U1.E2 (IO_L4P_T0_35)
- new net RDAL16: U1.U6 (IO_L16P_T2_34)
- new net RDAL17: U1.U3 (IO_L6P_T0_34)
- new net RDAL18: U1.T3 (IO_0_34)
- new net RDAL19: U1.R4 (IO_L13P_T2_MRCC_34)
- new net RDAL2: U1.L3 (IO_L14P_T2_SRCC_35)
- new net RDAL20: U1.L4 (IO_L18N_T2_35)
- new net RDAL21: U1.K1 (IO_L7P_T1_AD6P_35)
- new net RDAL3: U1.L5 (IO_L18P_T2_35)
- new net RDAL4: U1.K4 (IO_L13P_T2_MRCC_35)
- new net RDAL5: U1.K2 (IO_L9P_T1_DQS_AD7P_35)
- new net RDAL6: U1.J1 (IO_L7N_T1_AD6N_35)
- new net RDAL7: U1.K3 (IO_L14N_T2_SRCC_35)
- new net RDAL8: U1.G2 (IO_L8N_T1_AD14N_35)
- new net RDAL9: U1.H4 (IO_L12P_T1_MRCC_35)
- new net RWTBT: U1.U2 (IO_L2P_T0_34)
- new net TBS7: U1.W4 (IO_L12N_T1_MRCC_34)
- new net TDAL0: U1.V3 (IO_L6N_T0_VREF_34)
- new net TDAL1: U1.W2 (IO_L4P_T0_34)
- new net TDAL10: U1.D2 (IO_L4N_T0_35)
- new net TDAL11: U1.E3 (IO_L6N_T0_VREF_35)
- new net TDAL12: U1.B1 (IO_L1P_T0_AD4P_35)
- new net TDAL13: U1.C2 (IO_L2P_T0_AD12P_35)
- new net TDAL14: U1.A1 (IO_L1N_T0_AD4N_35)
- new net TDAL15: U1.B2 (IO_L2N_T0_AD12N_35)
- new net TDAL16: U1.Y2 (IO_L4N_T0_34)
- new net TDAL17: U1.AA1 (IO_L7P_T1_34)
- new net TDAL18: U1.V2 (IO_L2N_T0_34)
- new net TDAL19: U1.W1 (IO_L5P_T0_34)
- new net TDAL2: U1.J2 (IO_L9N_T1_DQS_AD7N_35)
- new net TDAL20: U1.K6 (IO_L17P_T2_35)
- new net TDAL21: U1.J4 (IO_L13N_T2_MRCC_35)
- new net TDAL3: U1.J5 (IO_L10P_T1_AD15P_35)
- new net TDAL4: U1.H2 (IO_L8P_T1_AD14P_35)
- new net TDAL5: U1.J6 (IO_L17N_T2_35)
- new net TDAL6: U1.G1 (IO_L5P_T0_AD13P_35)
- new net TDAL7: U1.H3 (IO_L11P_T1_SRCC_35)
- new net TDAL8: U1.F3 (IO_L6P_T0_35)
- new net TDAL9: U1.F4 (IO_0_35)
- new net TWTBT: U1.Y1 (IO_L5N_T0_34)
- no-connect marks 46 -> 11
Other:
- sheet I/O renamed IO
- sheet IO: file qbus.kicad_sch -> io.kicad_sch
- sheet QBUS: file qbus-2908.kicad_sch -> qbus.kicad_sch
- sheet QBUS ports: added RBS7, RDAL[0..21], RWTBT, TBS7, TDAL[0..21], TWTBT; removed ZBS7, ZDAL[0..21], ZWTBT, ~{RxDAL}, ~{TxDAL}
- moved on the sheet: C103, C104, C106, R104

Commit message: Switched the level converters to 74HCT2G04 and 75LVC2G04.  Still need to remap the FPGA pins to the signal odering.
Other:
- company: (none) -> Vintage Computer Enterprises
Changed lines of the file:
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@@
 	(title_block
 		(title "QSIC - QBUS Storage & I/O Card")
-		(date "2025-03-28")
+		(date "2025-04-12")
 		(rev "0.4")
-		(comment 1 "Clocks: RSYNC RDOUT RDMGI RDIN usb0_clk60")
+		(company "Vintage Computer Enterprises")
+		(comment 4 "Clocks: RSYNC RDOUT RDMGI RDIN usb0_clk60")
 	)
 	(text "QSIC - QBUS Storage & I/O Card"
